File: f411testingreliablitymotor/c2000_f280049_throttle/throttleecupcb/TasaruV0.0.1/TasaruV0.0.1.kicad_sch (KiCad schematic)
At the start: 162 parts, among them J1 Conn_02x05_Odd_EvenJtag, J2 173862-1, Q1 MMBT2222A, Q2 MMBT2222A, Q3 2N7002AQ, Q4 MMBT2222A, SW1 Push_Button, T1 MOT_PWM, T10 B_SPI_SIMO, T11 B_SPI_SOMI, T12 B_SPI_CLK, T13 B_SPI_CS, T14 +3v3, T2 MOT_PH, T3 +BATTP, T4 BRK_SENSE, T5 MOT_IPROPI2, T6 MOT_IPROPI1, T7 PGOOD, T8 CANTX, T9 CANRX, U1 SQJ147ELP-T1_GE3, U2 TPS1H100BQPWPRQ1, U3 DRV8873HPWPR, U4 F280049CPZS, U5 PSM33620S3QRDNRQ1, U6 SIT2024BA-S2-XXE-10.000000E, U7 PTCAN3404DRQ1, U8 AS5147U-HTSM, U9 TPS3702

Commit message: Tasaru V0.0.1 PCB: layout/schematic revisions, production outputs, docs
- Update KiCad schematic and PCB layout (major routing/schematic rework)
- Add production outputs: gerbers, BOM, fabrication toolkit config, freerouting DSN
- Add DRC/ERC reports and JLC DFM analysis
- Add LAYOUT.md and MCU_PIN_FUNCTION_MAP.md docs; update FIRMWARE_PIN_MAP.md and HANDOFF.md
- Add Hindsight logo/arrow footprint libraries and fp-lib-table
- Add component datasheets (LMR38020-Q1, TCAN3404-Q1, TPS3702-Q1, DRV8873 supplement)
- Prune old KiCad backup zips, add current ones; remove stale lock files
- Ignore .history/ editor cache, *.lck, and stray personal PDFs via .gitignore

Co-Authored-By: Claude Fable 5 <noreply@anthropic.com>
Parts:
- removed A5: SPARE_ADC_A5, TestPoint:TestPoint_THTPad_D2.0mm_Drill1.0mm, symbol Connector:TestPoint
- removed DZ1: BZT52C3V3S, PCM_Diode_SMD_AKL:D_SOD-323, symbol PCM_Diode_Zener_AKL:BZT52C3V3S
- removed IO17, IO18_X2, IO33: GPIO, PCM_SparkFun-Connector:TestPoint-0.75mm, symbol Connector:TestPoint
- removed Q1: MMBT2222A, PCM_Package_TO_SOT_SMD_AKL:SOT-23, symbol PCM_Transistor_BJT_AKL:MMBT2222A
- removed Q3: 2N7002AQ, PCM_Package_TO_SOT_SMD_AKL:SOT-23, symbol PCM_Transistor_MOSFET_AKL:2N7002AQ
- removed R_A5: 0.1mohm, PCM_Resistor_SMD_AKL:R_0201_0603Metric_Pad0.64x0.40mm_HandSolder, symbol PCM_Resistor_AKL:R_Generic
- removed U5: PSM33620S3QRDNRQ1, TPSM33620-Q1:RDN0011B-MFG, symbol TPSM33620-Q1:PSM33620S3QRDNRQ1
- added D1: BAV99R, PCM_Package_TO_SOT_SMD_AKL:SOT-23, symbol PCM_Diode_AKL:BAV99
- added L1: 10uH, PCM_SparkFun-Coil:Inductor_7.3x6.6mm, symbol PCM_SparkFun-Coil:6.8uH_7.3x6.6mm_4.5A
- added R34: 100k, PCM_Resistor_SMD_AKL:R_0603_1608Metric_Pad0.98x0.95mm_HandSolder, symbol PCM_Resistor_AKL:R_Generic
- added U5: PLMR38020FSQDDARQ1, lmr38020:DDA0008E-IPC_A, symbol lmr38020:PLMR38020FSQDDARQ1
- A2, A3, B3: footprint TestPoint:TestPoint_THTPad_D2.0mm_Drill1.0mm -> TestPoint:TestPoint_Pad_D1.5mm
- C14, C15: value 0.1uF -> 0.01uF
- C22, C24, C34: footprint Capacitor_THT:CP_Radial_D10.0mm_P5.00mm -> PCM_Capacitor_THT_US_AKL_Double:CP_Radial_D12.5mm_P5.00mm
- C32: value 10uF -> 22uF; footprint Capacitor_SMD:C_0805_2012Metric_Pad1.18x1.45mm_HandSolder -> Capacitor_SMD:C_1206_3216Metric_Pad1.33x1.80mm_HandSolder
- C33: value 10uF -> 0.1uF; footprint Capacitor_SMD:C_0805_2012Metric_Pad1.18x1.45mm_HandSolder -> Capacitor_SMD:C_1206_3216Metric_Pad1.33x1.80mm_HandSolder
- C35: value 0.1uF -> 4.7uF
- C37, C44: value 2.2uF -> 0.1uF
- D2: footprint PCM_Package_TO_SOT_SMD_AKL:SOT-23 -> PCM_Diode_SMD_AKL:D_SMB_TVS
- F2: footprint Fuse:Fuse_1206_3216Metric_Pad1.42x1.75mm_HandSolder -> PCM_Fuse_AKL:Fuseholder_Blade_Mini_Keystone_3568
- IO12: renamed from IO2; footprint PCM_SparkFun-Connector:TestPoint-0.75mm -> TestPoint:TestPoint_Pad_D1.0mm
- IO13, IO14, IO15, IO16, IO22_SW1, IO23_SW1, IO26, IO27, IO28, IO29, IO34, IO39, IO40: footprint PCM_SparkFun-Connector:TestPoint-0.75mm -> TestPoint:TestPoint_Pad_D1.0mm
- IO6: renamed from IO1; footprint PCM_SparkFun-Connector:TestPoint-0.75mm -> TestPoint:TestPoint_Pad_D1.0mm
- JP7: footprint Jumper:SolderJumper-2_P1.3mm_Open_RoundedPad1.0x1.5mm -> Jumper:SolderJumper-2_P1.3mm_Bridged2Bar_RoundedPad1.0x1.5mm
- R1, R15, R5: value 100k -> 10k; footprint PCM_Resistor_SMD_AKL:R_0201_0603Metric_Pad0.64x0.40mm_HandSolder -> PCM_Resistor_SMD_AKL:R_0402_1005Metric_Pad0.72x0.64mm_HandSolder
- R10, R11, R13, R14, R18, R20, R21, R22, R23, R24, R26, R28, R29, R3, R31, R32, R33, R4, R6, R8, R9, R_A2, R_A3, R_B3: footprint PCM_Resistor_SMD_AKL:R_0201_0603Metric_Pad0.64x0.40mm_HandSolder -> PCM_Resistor_SMD_AKL:R_0402_1005Metric_Pad0.72x0.64mm_HandSolder
- R12: value 100k -> 64.9k; footprint PCM_Resistor_SMD_AKL:R_0201_0603Metric_Pad0.64x0.40mm_HandSolder -> PCM_Resistor_SMD_AKL:R_0402_1005Metric_Pad0.72x0.64mm_HandSolder
- R16, R17, R19, R27, R30: footprint PCM_Resistor_SMD_AKL:R_0201_0603Metric_Pad0.64x0.40mm_HandSolder -> PCM_Resistor_SMD_AKL:R_0603_1608Metric_Pad0.98x0.95mm_HandSolder
- R2: value 22k -> 1k; footprint PCM_Resistor_SMD_AKL:R_0201_0603Metric_Pad0.64x0.40mm_HandSolder -> PCM_Resistor_SMD_AKL:R_0402_1005Metric_Pad0.72x0.64mm_HandSolder
- R25: value 100k -> 43.2k; footprint PCM_Resistor_SMD_AKL:R_0201_0603Metric_Pad0.64x0.40mm_HandSolder -> PCM_Resistor_SMD_AKL:R_0603_1608Metric_Pad0.98x0.95mm_HandSolder
- R7: value 22k -> 2.2k; footprint PCM_Resistor_SMD_AKL:R_0201_0603Metric_Pad0.64x0.40mm_HandSolder -> PCM_Resistor_SMD_AKL:R_0402_1005Metric_Pad0.72x0.64mm_HandSolder
- T10: value B_SPI_SIMO -> A_SPI_SIMO
- T11: value B_SPI_SOMI -> A_SPI_CLK
- T12: value B_SPI_CLK -> A_SPI_SOMI
- T13: value B_SPI_CS -> A_SPI_CS
Connections:
- net +3V3: now also C45.2, C46.2, R33.1, U8.11 (VDD), U8.12 (VDD3V3), D1.1 (A), L1.2, R34.1
- net +BATT: no longer U1.2 (S), U1.3 (S)
- net +SOL: now also J2.6; no longer J2.16
- net 12V_BRAKEIN: no longer R2.2
- net BRK_SENSE: now also R2.2, D1.3 (C); no longer JP9.1 (A)
- net BRK_SW: now also Q4.3 (C), R33.2; no longer R33.1
- net DISABLE: now also R11.2, R5.1; no longer R14.2
- net GND: now also R25.2, U3.EPAD, D1.2 (K), U5.1 (GND), U5.9 (EP); no longer C37.1
- net MOT_DISABLE: now also U4.75 (GPIO04); no longer U4.97 (GPIO06)
- net MOT_IPROPI1: now also T6.1, U4.23 (A0_B15_C15_DACA_OUT); no longer U3.10 (IPROPI1)
- net MOT_IPROPI2: now also T5.1, U4.41 (B0); no longer U3.12 (IPROPI2)
- net MOT_OUT+: now also J2.15, J2.16; no longer J2.4, J2.6
- net MOT_OUT-: now also J2.4; no longer J2.15
- net MOT_nSLEEP: now also U4.76 (GPIO03); no longer U4.89 (GPIO05)
- net PGOOD: now also U4.53 (GPIO33), R34.2, U5.6 (PG); no longer R25.1
- net SENSOR_PWM: now also U4.89 (GPIO05); no longer U4.75 (GPIO04)
- net SPI_CLK: now also U4.67 (GPIO58); no longer U4.90 (GPIO09)
- net SPI_CS: now also U4.92 (GPIO59); no longer U4.52 (GPIO11)
- net SPI_MISO: now also U4.66 (GPIO57); no longer U4.93 (GPIO10)
- net SPI_MOSI: now also U4.65 (GPIO56); no longer U4.74 (GPIO08)
- net nFault: now also U4.78 (GPIO01); no longer U4.51 (GPIO12)
- net Vin: now reaches C22.1, C24.1, C32.2, C33.2, C35.2, F1.2
- net Vin: now also U5.2 (EN), U5.3 (VIN)
- net at C37.2: now also U5.7 (BOOT); no longer R25.2
- net at R12.1: now also U5.4 (RT_SYNC); no longer R11.2
- net 10Mhz_Ocillator_Out: now reaches U4.69 (X1), U6.5 (OUT)
- net at R2.1: now also JP9.1 (A); no longer R5.1
- net SOL_CLEAN_GND: now reaches D4.1 (A), R13.1, R18.2, U2.15 (PAD), U2.2 (GND)
- net at IO12.1: now also U4.51 (GPIO12); no longer U4.76 (GPIO03)
- net 15aFusedBATT: now reaches F2.1, U1.1 (S)
- net 15aFusedBATT: now also U1.2 (S), U1.3 (S)
- net at IO6.1: now also U4.97 (GPIO06); no longer U4.78 (GPIO01)
- net A5: no longer names the net of U4.35 (A5)
- net B_SPI_CLK renamed A_SPI_SOMI
- net A_SPI_SOMI: now also U4.93 (GPIO10); no longer U4.67 (GPIO58)
- net B_SPI_CS renamed A_SPI_CS
- net A_SPI_CS: now also U4.52 (GPIO11); no longer U4.92 (GPIO59)
- net B_SPI_SIMO renamed A_SPI_SIMO
- net A_SPI_SIMO: now also U4.74 (GPIO08); no longer U4.65 (GPIO56)
- net B_SPI_SOMI renamed A_SPI_CLK
- net A_SPI_CLK: now also U4.90 (GPIO09); no longer U4.66 (GPIO57)
- new net: R14.2, R25.1, U5.5 (FB)
- new net: C37.1, L1.1, U5.8 (SW)
- new net: JP11.2 (B), U3.10 (IPROPI1)
- new net: JP12.2 (B), U3.12 (IPROPI2)
Other:
- note added: "Enable SOL"
- note added: "Place Near U4"
- note added: "Sets IN to LOW to disable Sol when brake is pressed"
- moved on the sheet: C22, C24, C42, C43, D2, D3, D4, F1, F2, IO12, IO6, JP11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
